File: integrator.sch (KiCad schematic (older format))
At the start: 4 parts, among them U4 MCP6004, U5 SN74LVC1G3157

Commit message: Rev A
Connections:
- net INT_FB: now also U4.2 (-); no longer U4.9 (-)
- net VOUT: now also U4.1; no longer U4.8
- net VREF: now also U4.3 (+); no longer U4.10 (+)
Changed lines of the file:
@@
 $Comp
 L MCP6004 U4
-U 3 1 59C031BE
+U 1 1 59C031BE
 P 3100 2500
 AR Path="/59C031A5/59C031BE" Ref="U4"  Part="1"
@@
 F 2 "olof:SOIC-14_3.9x8.7mm_Pitch1.27mm" H 3050 2600 50  0001 C CNN
 F 3 "" H 3150 2700 50  0000 C CNN
-	3    3100 2500
+	1    3100 2500
 	1    0    0    -1
 $EndComp
@@
 AR Path="/59C0659A/59C03233" Ref="R42"  Part="1"
 AR Path="/59C065F7/59C03233" Ref="R43"  Part="1"
-F 0 "R43" V 2530 2600 50  0000 C CNN
+F 0 "R40" V 2530 2600 50  0000 C CNN
 F 1 "6M8" V 2450 2600 50  0000 C CNN
 F 2 "olof:R_0805_HandSoldering" V 2380 2600 50  0001 C CNN
@@
 AR Path="/59C0659A/59C03273" Ref="#PWR076"  Part="1"
 AR Path="/59C065F7/59C03273" Ref="#PWR080"  Part="1"
-F 0 "#PWR080" H 3000 2000 50  0001 C CNN
+F 0 "#PWR068" H 3000 2000 50  0001 C CNN
 F 1 "VCC" H 3000 2300 50  0000 C CNN
 F 2 "" H 3000 2150 50  0000 C CNN
@@
 AR Path="/59C0659A/59C0328B" Ref="#PWR077"  Part="1"
 AR Path="/59C065F7/59C0328B" Ref="#PWR081"  Part="1"
-F 0 "#PWR081" H 3000 2600 50  0001 C CNN
+F 0 "#PWR069" H 3000 2600 50  0001 C CNN
 F 1 "GND" H 3000 2700 50  0000 C CNN
 F 2 "" H 3000 2850 50  0000 C CNN
@@
 AR Path="/59C0659A/59C032B2" Ref="C12"  Part="1"
 AR Path="/59C065F7/59C032B2" Ref="C13"  Part="1"
-F 0 "C13" H 3025 3350 50  0000 L CNN
+F 0 "C10" H 3025 3350 50  0000 L CNN
 F 1 "220n" H 3025 3150 50  0000 L CNN
 F 2 "olof:C_0805_HandSoldering" H 3038 3100 50  0001 C CNN
@@
 AR Path="/59C0659A/5A0B5EBF" Ref="U7"  Part="1"
 AR Path="/59C065F7/5A0B5EBF" Ref="U8"  Part="1"
-F 0 "U8" H 2850 4000 60  0000 C CNN
+F 0 "U5" H 2850 4000 60  0000 C CNN
 F 1 "SN74LVC1G3157" H 3550 4000 60  0000 C CNN
 F 2 "TO_SOT_Packages_SMD:SOT-23-6" H 3050 4300 60  0001 C CNN
@@
 AR Path="/59C0659A/5A0B5F36" Ref="#PWR078"  Part="1"
 AR Path="/59C065F7/5A0B5F36" Ref="#PWR082"  Part="1"
-F 0 "#PWR082" H 3050 3650 50  0001 C CNN
+F 0 "#PWR070" H 3050 3650 50  0001 C CNN
 F 1 "VCC" H 3050 3950 50  0000 C CNN
 F 2 "" H 3050 3800 50  0000 C CNN
@@
 AR Path="/59C0659A/5A0B5F64" Ref="#PWR079"  Part="1"
 AR Path="/59C065F7/5A0B5F64" Ref="#PWR083"  Part="1"
-F 0 "#PWR083" H 3050 4500 50  0001 C CNN
+F 0 "#PWR071" H 3050 4500 50  0001 C CNN
 F 1 "GND" H 3050 4600 50  0000 C CNN
 F 2 "" H 3050 4750 50  0000 C CNN

Commit message: Added 5V regulator
Parts:
- C10: value 220n -> 100n
Connections:
- net INT_FB: now also U4.9 (-); no longer U4.2 (-)
- net VOUT: now also U4.8; no longer U4.1
- net VREF: now also U4.10 (+); no longer U4.3 (+)
Changed lines of the file:
@@
 $Descr A4 11693 8268
 encoding utf-8
-Sheet 7 10
+Sheet 8 11
 Title ""
 Date ""
@@
 $Comp
 L MCP6004 U4
-U 1 1 59C031BE
+U 3 1 59C031BE
 P 3100 2500
 AR Path="/59C031A5/59C031BE" Ref="U4"  Part="1"
@@
 F 2 "olof:SOIC-14_3.9x8.7mm_Pitch1.27mm" H 3050 2600 50  0001 C CNN
 F 3 "" H 3150 2700 50  0000 C CNN
-	1    3100 2500
+	3    3100 2500
 	1    0    0    -1
 $EndComp
@@
 AR Path="/59C0659A/59C03233" Ref="R42"  Part="1"
 AR Path="/59C065F7/59C03233" Ref="R43"  Part="1"
-F 0 "R40" V 2530 2600 50  0000 C CNN
+F 0 "R43" V 2530 2600 50  0000 C CNN
 F 1 "6M8" V 2450 2600 50  0000 C CNN
 F 2 "olof:R_0805_HandSoldering" V 2380 2600 50  0001 C CNN
@@
 $EndComp
 $Comp
-L VCC #PWR068
+L VCC #PWR051
 U 1 1 59C03273
 P 3000 2150
-AR Path="/59C031A5/59C03273" Ref="#PWR068"  Part="1"
-AR Path="/59C0653D/59C03273" Ref="#PWR072"  Part="1"
-AR Path="/59C0659A/59C03273" Ref="#PWR076"  Part="1"
-AR Path="/59C065F7/59C03273" Ref="#PWR080"  Part="1"
-F 0 "#PWR068" H 3000 2000 50  0001 C CNN
+AR Path="/59C031A5/59C03273" Ref="#PWR051"  Part="1"
+AR Path="/59C0653D/59C03273" Ref="#PWR055"  Part="1"
+AR Path="/59C0659A/59C03273" Ref="#PWR059"  Part="1"
+AR Path="/59C065F7/59C03273" Ref="#PWR063"  Part="1"
+F 0 "#PWR063" H 3000 2000 50  0001 C CNN
 F 1 "VCC" H 3000 2300 50  0000 C CNN
 F 2 "" H 3000 2150 50  0000 C CNN
@@
 $EndComp
 $Comp
-L GND #PWR069
+L GND #PWR052
 U 1 1 59C0328B
 P 3000 2850
-AR Path="/59C031A5/59C0328B" Ref="#PWR069"  Part="1"
-AR Path="/59C0653D/59C0328B" Ref="#PWR073"  Part="1"
-AR Path="/59C0659A/59C0328B" Ref="#PWR077"  Part="1"
-AR Path="/59C065F7/59C0328B" Ref="#PWR081"  Part="1"
-F 0 "#PWR069" H 3000 2600 50  0001 C CNN
+AR Path="/59C031A5/59C0328B" Ref="#PWR052"  Part="1"
+AR Path="/59C0653D/59C0328B" Ref="#PWR056"  Part="1"
+AR Path="/59C0659A/59C0328B" Ref="#PWR060"  Part="1"
+AR Path="/59C065F7/59C0328B" Ref="#PWR064"  Part="1"
+F 0 "#PWR064" H 3000 2600 50  0001 C CNN
 F 1 "GND" H 3000 2700 50  0000 C CNN
 F 2 "" H 3000 2850 50  0000 C CNN
@@
 AR Path="/59C0659A/59C032B2" Ref="C12"  Part="1"
 AR Path="/59C065F7/59C032B2" Ref="C13"  Part="1"
-F 0 "C10" H 3025 3350 50  0000 L CNN
-F 1 "220n" H 3025 3150 50  0000 L CNN
+F 0 "C13" H 3025 3350 50  0000 L CNN
+F 1 "100n" H 3025 3150 50  0000 L CNN
 F 2 "olof:C_0805_HandSoldering" H 3038 3100 50  0001 C CNN
 F 3 "" H 3000 3250 50  0000 C CNN
@@
 AR Path="/59C0659A/5A0B5EBF" Ref="U7"  Part="1"
 AR Path="/59C065F7/5A0B5EBF" Ref="U8"  Part="1"
-F 0 "U5" H 2850 4000 60  0000 C CNN
+F 0 "U8" H 2850 4000 60  0000 C CNN
 F 1 "SN74LVC1G3157" H 3550 4000 60  0000 C CNN
 F 2 "TO_SOT_Packages_SMD:SOT-23-6" H 3050 4300 60  0001 C CNN
@@
 $EndComp
 $Comp
-L VCC #PWR070
+L VCC #PWR053
 U 1 1 5A0B5F36
 P 3050 3800
-AR Path="/59C031A5/5A0B5F36" Ref="#PWR070"  Part="1"
-AR Path="/59C0653D/5A0B5F36" Ref="#PWR074"  Part="1"
-AR Path="/59C0659A/5A0B5F36" Ref="#PWR078"  Part="1"
-AR Path="/59C065F7/5A0B5F36" Ref="#PWR082"  Part="1"
-F 0 "#PWR070" H 3050 3650 50  0001 C CNN
+AR Path="/59C031A5/5A0B5F36" Ref="#PWR053"  Part="1"
+AR Path="/59C0653D/5A0B5F36" Ref="#PWR057"  Part="1"
+AR Path="/59C0659A/5A0B5F36" Ref="#PWR061"  Part="1"
+AR Path="/59C065F7/5A0B5F36" Ref="#PWR065"  Part="1"
+F 0 "#PWR065" H 3050 3650 50  0001 C CNN
 F 1 "VCC" H 3050 3950 50  0000 C CNN
 F 2 "" H 3050 3800 50  0000 C CNN
@@
 	3050 3800 3050 3850
 $Comp
-L GND #PWR071
+L GND #PWR054
 U 1 1 5A0B5F64
 P 3050 4750
-AR Path="/59C031A5/5A0B5F64" Ref="#PWR071"  Part="1"
-AR Path="/59C0653D/5A0B5F64" Ref="#PWR075"  Part="1"
-AR Path="/59C0659A/5A0B5F64" Ref="#PWR079"  Part="1"
-AR Path="/59C065F7/5A0B5F64" Ref="#PWR083"  Part="1"
-F 0 "#PWR071" H 3050 4500 50  0001 C CNN
+AR Path="/59C031A5/5A0B5F64" Ref="#PWR054"  Part="1"
+AR Path="/59C0653D/5A0B5F64" Ref="#PWR058"  Part="1"
+AR Path="/59C0659A/5A0B5F64" Ref="#PWR062"  Part="1"
+AR Path="/59C065F7/5A0B5F64" Ref="#PWR066"  Part="1"
+F 0 "#PWR066" H 3050 4500 50  0001 C CNN
 F 1 "GND" H 3050 4600 50  0000 C CNN
 F 2 "" H 3050 4750 50  0000 C CNN

Commit message: Removed 0R resistors and started new layout
Connections:
- net INT_FB: now also U4.13 (-); no longer U4.9 (-)
- net VOUT: now also U4.14; no longer U4.8
- net VREF: now also U4.12 (+); no longer U4.10 (+)
Changed lines of the file:
@@
 $Comp
 L MCP6004 U4
-U 3 1 59C031BE
+U 4 1 59C031BE
 P 3100 2500
 AR Path="/59C031A5/59C031BE" Ref="U4"  Part="1"
@@
 F 2 "olof:SOIC-14_3.9x8.7mm_Pitch1.27mm" H 3050 2600 50  0001 C CNN
 F 3 "" H 3150 2700 50  0000 C CNN
-	3    3100 2500
+	4    3100 2500
 	1    0    0    -1
 $EndComp
@@
 AR Path="/59C0659A/59C03233" Ref="R42"  Part="1"
 AR Path="/59C065F7/59C03233" Ref="R43"  Part="1"
-F 0 "R43" V 2530 2600 50  0000 C CNN
+F 0 "R42" V 2530 2600 50  0000 C CNN
 F 1 "6M8" V 2450 2600 50  0000 C CNN
 F 2 "olof:R_0805_HandSoldering" V 2380 2600 50  0001 C CNN
@@
 $EndComp
 $Comp
-L VCC #PWR051
+L VCC #PWR061
 U 1 1 59C03273
 P 3000 2150
-AR Path="/59C031A5/59C03273" Ref="#PWR051"  Part="1"
-AR Path="/59C0653D/59C03273" Ref="#PWR055"  Part="1"
-AR Path="/59C0659A/59C03273" Ref="#PWR059"  Part="1"
-AR Path="/59C065F7/59C03273" Ref="#PWR063"  Part="1"
-F 0 "#PWR063" H 3000 2000 50  0001 C CNN
+AR Path="/59C031A5/59C03273" Ref="#PWR061"  Part="1"
+AR Path="/59C0653D/59C03273" Ref="#PWR065"  Part="1"
+AR Path="/59C0659A/59C03273" Ref="#PWR069"  Part="1"
+AR Path="/59C065F7/59C03273" Ref="#PWR073"  Part="1"
+F 0 "#PWR073" H 3000 2000 50  0001 C CNN
 F 1 "VCC" H 3000 2300 50  0000 C CNN
 F 2 "" H 3000 2150 50  0000 C CNN
@@
 $EndComp
 $Comp
-L GND #PWR052
+L GND #PWR062
 U 1 1 59C0328B
 P 3000 2850
-AR Path="/59C031A5/59C0328B" Ref="#PWR052"  Part="1"
-AR Path="/59C0653D/59C0328B" Ref="#PWR056"  Part="1"
-AR Path="/59C0659A/59C0328B" Ref="#PWR060"  Part="1"
-AR Path="/59C065F7/59C0328B" Ref="#PWR064"  Part="1"
-F 0 "#PWR064" H 3000 2600 50  0001 C CNN
+AR Path="/59C031A5/59C0328B" Ref="#PWR062"  Part="1"
+AR Path="/59C0653D/59C0328B" Ref="#PWR066"  Part="1"
+AR Path="/59C0659A/59C0328B" Ref="#PWR070"  Part="1"
+AR Path="/59C065F7/59C0328B" Ref="#PWR074"  Part="1"
+F 0 "#PWR074" H 3000 2600 50  0001 C CNN
 F 1 "GND" H 3000 2700 50  0000 C CNN
 F 2 "" H 3000 2850 50  0000 C CNN
@@
 AR Path="/59C0659A/59C032B2" Ref="C12"  Part="1"
 AR Path="/59C065F7/59C032B2" Ref="C13"  Part="1"
-F 0 "C13" H 3025 3350 50  0000 L CNN
+F 0 "C12" H 3025 3350 50  0000 L CNN
 F 1 "100n" H 3025 3150 50  0000 L CNN
 F 2 "olof:C_0805_HandSoldering" H 3038 3100 50  0001 C CNN
@@
 AR Path="/59C0659A/5A0B5EBF" Ref="U7"  Part="1"
 AR Path="/59C065F7/5A0B5EBF" Ref="U8"  Part="1"
-F 0 "U8" H 2850 4000 60  0000 C CNN
+F 0 "U7" H 2850 4000 60  0000 C CNN
 F 1 "SN74LVC1G3157" H 3550 4000 60  0000 C CNN
 F 2 "TO_SOT_Packages_SMD:SOT-23-6" H 3050 4300 60  0001 C CNN
@@
 $EndComp
 $Comp
-L VCC #PWR053
+L VCC #PWR063
 U 1 1 5A0B5F36
 P 3050 3800
-AR Path="/59C031A5/5A0B5F36" Ref="#PWR053"  Part="1"
-AR Path="/59C0653D/5A0B5F36" Ref="#PWR057"  Part="1"
-AR Path="/59C0659A/5A0B5F36" Ref="#PWR061"  Part="1"
-AR Path="/59C065F7/5A0B5F36" Ref="#PWR065"  Part="1"
-F 0 "#PWR065" H 3050 3650 50  0001 C CNN
+AR Path="/59C031A5/5A0B5F36" Ref="#PWR063"  Part="1"
+AR Path="/59C0653D/5A0B5F36" Ref="#PWR067"  Part="1"
+AR Path="/59C0659A/5A0B5F36" Ref="#PWR071"  Part="1"
+AR Path="/59C065F7/5A0B5F36" Ref="#PWR075"  Part="1"
+F 0 "#PWR075" H 3050 3650 50  0001 C CNN
 F 1 "VCC" H 3050 3950 50  0000 C CNN
 F 2 "" H 3050 3800 50  0000 C CNN
@@
 	3050 3800 3050 3850
 $Comp
-L GND #PWR054
+L GND #PWR064
 U 1 1 5A0B5F64
 P 3050 4750
-AR Path="/59C031A5/5A0B5F64" Ref="#PWR054"  Part="1"
-AR Path="/59C0653D/5A0B5F64" Ref="#PWR058"  Part="1"
-AR Path="/59C0659A/5A0B5F64" Ref="#PWR062"  Part="1"
-AR Path="/59C065F7/5A0B5F64" Ref="#PWR066"  Part="1"
-F 0 "#PWR066" H 3050 4500 50  0001 C CNN
+AR Path="/59C031A5/5A0B5F64" Ref="#PWR064"  Part="1"
+AR Path="/59C0653D/5A0B5F64" Ref="#PWR068"  Part="1"
+AR Path="/59C0659A/5A0B5F64" Ref="#PWR072"  Part="1"
+AR Path="/59C065F7/5A0B5F64" Ref="#PWR076"  Part="1"
+F 0 "#PWR076" H 3050 4500 50  0001 C CNN
 F 1 "GND" H 3050 4600 50  0000 C CNN
 F 2 "" H 3050 4750 50  0000 C CNN
