File: servo-joystick.kicad_pcb (KiCad board)
At the start: 2 copper layers, 100 x 80 mm, 114 parts, among them P1 CONN_01X02, P2 CONN_01X03, P3 CONN_01X03, P4 CONN_01X03, P5 CONN_01X03, U1 MCP6002, U2 MCP6004, U3 MCP6004, U4 MCP6004, U5 SN74LVC1G3157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

Commit message: Correct pinout for LD2981
Parts:
- turned C22 to 180 degrees
Connections:
- U9 pad 4: VCC -> Net-(U9-Pad4)
- U9 pad 5: Net-(U9-Pad5) -> VCC
Changed lines of the file:
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@@
   (net 86 "/PWM #4/BUF")
   (net 87 +6V)
-  (net 88 "Net-(U9-Pad5)")
+  (net 88 "Net-(U9-Pad4)")
   (net_class Default "This is the default net class."
     (clearance 0.24)
@@
     (add_net "Net-(U7-Pad3)")
     (add_net "Net-(U8-Pad3)")
-    (add_net "Net-(U9-Pad5)")
+    (add_net "Net-(U9-Pad4)")
     (add_net "Net-(VR1-Pad11)")
     (add_net "Net-(VR1-Pad12)")
@@
   )
   (module olof:C_0805_HandSoldering (layer F.Cu)
-    (at 118.5 116.5)
+    (at 118.49 116.49 180)
     (descr "Capacitor SMD 0805, hand soldering")
     (tags "capacitor 0805")
     (attr smd)
-    (fp_text reference C22 (at 3.048 0 90) (layer F.SilkS)
+    (fp_text reference C22 (at -3 -0.01 270) (layer F.SilkS)
       (effects (font (size 0.75 0.75) (thickness 0.11)))
     )
-    (fp_text value 2u2 (at 0 2.1) (layer F.Fab)
+    (fp_text value 2u2 (at 0 2.1 180) (layer F.Fab)
       (effects (font (size 1 1) (thickness 0.15)))
     )
@@
     (fp_line (start 0.5 -0.85) (end -0.5 -0.85) (layer F.SilkS) (width 0.15))
     (fp_line (start -0.5 0.85) (end 0.5 0.85) (layer F.SilkS) (width 0.15))
-    (pad 1 smd rect (at -1.25 0) (size 1.5 1.25) (layers F.Cu F.Paste F.Mask)
+    (pad 1 smd rect (at -1.25 0 180) (size 1.5 1.25) (layers F.Cu F.Paste F.Mask)
       (net 1 VCC))
-    (pad 2 smd rect (at 1.25 0) (size 1.5 1.25) (layers F.Cu F.Paste F.Mask)
+    (pad 2 smd rect (at 1.25 0 180) (size 1.5 1.25) (layers F.Cu F.Paste F.Mask)
       (net 2 GND))
     (model Capacitors_SMD.3dshapes/C_0805_HandSoldering.wrl
@@
     (tags SOT-23-5)
     (attr smd)
-    (fp_text reference U9 (at 3.1 0 360) (layer F.SilkS)
+    (fp_text reference U9 (at 1.53 -2.81 360) (layer F.SilkS)
       (effects (font (size 1 1) (thickness 0.15)))
     )
@@
       (net 87 +6V))
     (pad 4 smd rect (at 1.3 0.95 270) (size 1.46 0.65) (layers F.Cu F.Paste F.Mask)
-      (net 1 VCC))
+      (net 88 "Net-(U9-Pad4)"))
     (pad 5 smd rect (at 1.3 -0.95 270) (size 1.46 0.65) (layers F.Cu F.Paste F.Mask)
-      (net 88 "Net-(U9-Pad5)"))
+      (net 1 VCC))
     (model TO_SOT_Packages_SMD.3dshapes/SOT-23-5.wrl
       (at (xyz 0 0 0))
@@
     (arrow2b (pts (xy 24.953179 174.322574) (xy 26.079683 173.736153)))
   )
+  (segment (start 119.45 114.93) (end 119.74 115.22) (width 0.25) (layer F.Cu) (net 1))
+  (segment (start 119.74 115.22) (end 119.74 116.49) (width 0.25) (layer F.Cu) (net 1))
+  (segment (start 119.45 113.8) (end 119.45 114.93) (width 0.25) (layer F.Cu) (net 1))
   (segment (start 109.625 152) (end 109.625 151.625) (width 0.25) (layer F.Cu) (net 1))
   (segment (start 26.75 132.875) (end 27.125 132.875) (width 0.25) (layer F.Cu) (net 1))
@@
   (segment (start 113.875 153.75) (end 115 152.625) (width 0.25) (layer F.Cu) (net 1))
   (segment (start 115 152.625) (end 115 151.25) (width 0.25) (layer F.Cu) (net 1))
-  (segment (start 117.55 113.8) (end 117.55 115.05) (width 0.25) (layer F.Cu) (net 1))
-  (segment (start 117.55 115.05) (end 117.25 115.35) (width 0.25) (layer F.Cu) (net 1))
-  (segment (start 117.25 115.35) (end 117.25 116.5) (width 0.25) (layer F.Cu) (net 1))
   (segment (start 61.2 131.25) (end 59.6 131.25) (width 0.25) (layer F.Cu) (net 1))
   (segment (start 59.6 131.25) (end 58.45 130.1) (width 0.25) (layer F.Cu) (net 1))
@@
   (segment (start 93.75 108) (end 93.75 105.2) (width 0.25) (layer F.Cu) (net 1))
   (segment (start 56.25 105.2) (end 56.25 108) (width 0.25) (layer F.Cu) (net 1))
+  (segment (start 115.6 116.49) (end 115.6 121.68) (width 0.25) (layer B.Cu) (net 2))
+  (segment (start 115.6 121.68) (end 116.375 122.455) (width 0.25) (layer B.Cu) (net 2))
+  (segment (start 116.375 122.455) (end 116.375 127.875) (width 0.25) (layer B.Cu) (net 2))
+  (segment (start 115.6 116.49) (end 115.6 115.4) (width 0.25) (layer B.Cu) (net 2))
+  (segment (start 115.6 115.4) (end 118.5 112.5) (width 0.25) (layer B.Cu) (net 2))
+  (segment (start 117.24 116.49) (end 115.6 116.49) (width 0.25) (layer F.Cu) (net 2))
+  (via (at 115.6 116.49) (size 0.6) (drill 0.4) (layers F.Cu B.Cu) (net 2))
   (segment (start 30.375 132.875) (end 30.75 132.875) (width 0.25) (layer F.Cu) (net 2))
   (segment (start 26.75 137.125) (end 27.125 137.125) (width 0.25) (layer F.Cu) (net 2))
@@
   (segment (start 115.9 108.5) (end 116.324264 108.5) (width 0.25) (layer B.Cu) (net 2))
   (segment (start 116.324264 108.5) (end 117.25 108.5) (width 0.25) (layer B.Cu) (net 2))
-  (segment (start 119.55 116.5) (end 118.5 115.45) (width 0.25) (layer B.Cu) (net 2))
-  (segment (start 118.5 115.45) (end 118.5 114.75) (width 0.25) (layer B.Cu) (net 2))
-  (segment (start 121.2 116.5) (end 119.55 116.5) (width 0.25) (layer B.Cu) (net 2))
-  (segment (start 119.75 116.5) (end 121.2 116.5) (width 0.25) (layer F.Cu) (net 2))
-  (via (at 121.2 116.5) (size 0.6) (drill 0.4) (layers F.Cu B.Cu) (net 2))
   (segment (start 117.25 108.5) (end 115.9 108.5) (width 0.25) (layer F.Cu) (net 2))
   (via (at 115.9 108.5) (size 0.6) (drill 0.4) (layers F.Cu B.Cu) (net 2))
@@
   (segment (start 120 103) (end 121.5 103) (width 0.25) (layer B.Cu) (net 2))
   (segment (start 121.5 103) (end 119.25 103) (width 0.25) (layer B.Cu) (net 2))
-  (segment (start 118.5 112.5) (end 118.5 114.75) (width 0.25) (layer B.Cu) (net 2))
   (segment (start 117.25 109) (end 118.5 110.25) (width 0.25) (layer B.Cu) (net 2))
   (segment (start 118.5 110.25) (end 118.5 112.5) (width 0.25) (layer B.Cu) (net 2))
@@
   (segment (start 74.5 88.25) (end 76 88.25) (width 0.25) (layer F.Cu) (net 2))
   (via (at 76 88.25) (size 0.6) (drill 0.4) (layers F.Cu B.Cu) (net 2))
-  (segment (start 116.375 127.875) (end 116.375 116.875) (width 0.25) (layer B.Cu) (net 2))
   (segment (start 52.25 124) (end 53.7 124) (width 0.25) (layer F.Cu) (net 2))
   (segment (start 53.7 124) (end 53.75 123.95) (width 0.25) (layer F.Cu) (net 2))
